File: GreenhouseController/ILI9341.sch (KiCad schematic (older format))
At the start: 1 part

Commit message: Connect my schematic to stm32 board
Parts:
- U?: symbol Driver_Display:ili9341-new -> GreenhouseController-rescue:ili9341-new-Driver_Display
Changed lines of the file:
@@
 VSS(18)
 $Comp
-L Driver_Display:ili9341-new U?
+L GreenhouseController-rescue:ili9341-new-Driver_Display U?
 U 1 1 61964760
 P 5800 3050
