File: GreenhouseController/NUCLEO.sch (KiCad schematic (older format))
At the start: 6 parts

Commit message: Connect my schematic to stm32 board
Parts:
- U? (x6): symbol NUCLEO-F410RB:NUCLEO-F410RB -> GreenhouseController-rescue:NUCLEO-F410RB-NUCLEO-F410RB
Connections:
- net labels added: ADC_IN0(PA1)
- wire segments 0 -> 1
Changed lines of the file:
@@
 $EndDescr
 $Comp
-L NUCLEO-F410RB:NUCLEO-F410RB U?
+L GreenhouseController-rescue:NUCLEO-F410RB-NUCLEO-F410RB U?
 U 1 1 61938EA9
 P 2200 2550
@@
 $EndComp
 $Comp
-L NUCLEO-F410RB:NUCLEO-F410RB U?
+L GreenhouseController-rescue:NUCLEO-F410RB-NUCLEO-F410RB U?
 U 2 1 6193B543
 P 4400 2550
@@
 $EndComp
 $Comp
-L NUCLEO-F410RB:NUCLEO-F410RB U?
+L GreenhouseController-rescue:NUCLEO-F410RB-NUCLEO-F410RB U?
 U 3 1 6193DFBD
 P 6500 2000
@@
 $EndComp
 $Comp
-L NUCLEO-F410RB:NUCLEO-F410RB U?
+L GreenhouseController-rescue:NUCLEO-F410RB-NUCLEO-F410RB U?
 U 4 1 619400A3
 P 8450 2050
@@
 $EndComp
 $Comp
-L NUCLEO-F410RB:NUCLEO-F410RB U?
+L GreenhouseController-rescue:NUCLEO-F410RB-NUCLEO-F410RB U?
 U 5 1 61941A55
 P 2100 5700
@@
 $EndComp
 $Comp
-L NUCLEO-F410RB:NUCLEO-F410RB U?
+L GreenhouseController-rescue:NUCLEO-F410RB-NUCLEO-F410RB U?
 U 6 1 6194455B
 P 4200 5600
@@
 	1    0    0    -1
 $EndComp
+Text GLabel 1100 2150 0    50   Input ~ 0
+ADC_IN0(PA1)
+Wire Wire Line
+	1500 2150 1100 2150
 $EndSCHEMATC
